File: Hard/PM_Board.sch (KiCad schematic (older format))
At the start: 76 parts, among them J1 Micro_SD_Card_Det_Hirose_DM3AT, J101 LiPo_V+, J102 LiPo_V-, J2 KRC_Conn_SWD, J3 USB_B_Micro, J4 KRC_Conn_CAN, J5 KRC_Conn_CAN, J6 Umbilical, J7 SW, Q1 SSM3J328R, Q2 2n7002, Q3 SSM3J328R, U1 CY8C58xxLTI-LPxxx, U2 INA226, U3 NCV7342, Y1 24MHz

Commit message: [update] READMEを整備
Parts:
- D6, D7, D8, J1, Q2: Agency 秋月電子 -> akizuki
Changed lines of the file:
@@
 F 2 "Package_TO_SOT_SMD:SOT-23" H 2850 5750 50  0001 C CNN
 F 3 "http://akizukidenshi.com/download/2n7002.pdf" H 2650 5650 50  0001 C CNN
-F 4 "秋月電子" H 200 0   50  0001 C CNN "Agency"
+F 4 "akizuki" H 200 0   50  0001 C CNN "Agency"
 F 5 "http://akizukidenshi.com/catalog/g/gI-03919/" H 200 0   50  0001 C CNN "Link"
 F 6 "2N7002" H 200 0   50  0001 C CNN "MPN"
@@
 F 2 "Diode_SMD:D_TUMD2" V 2900 2350 50  0001 C CNN
 F 3 "http://akizukidenshi.com/download/ds/rohm/rsx101vam30-j.pdf" V 2900 2350 50  0001 C CNN
-F 4 "秋月電子" H 2900 2350 50  0001 C CNN "Agency"
+F 4 "akizuki" H 2900 2350 50  0001 C CNN "Agency"
 F 5 "http://akizukidenshi.com/catalog/g/gI-05951/" H 2900 2350 50  0001 C CNN "Link"
 F 6 "RSX101VAM-30TR" H 2900 2350 50  0001 C CNN "MPN"
@@
 F 2 "Diode_SMD:D_TUMD2" V 2900 3350 50  0001 C CNN
 F 3 "http://akizukidenshi.com/download/ds/rohm/rsx101vam30-j.pdf" V 2900 3350 50  0001 C CNN
-F 4 "秋月電子" H 2900 3350 50  0001 C CNN "Agency"
+F 4 "akizuki" H 2900 3350 50  0001 C CNN "Agency"
 F 5 "http://akizukidenshi.com/catalog/g/gI-05951/" H 2900 3350 50  0001 C CNN "Link"
 F 6 "RSX101VAM-30TR" H 2900 3350 50  0001 C CNN "MPN"
@@
 F 2 "Connector_Card:microSD_HC_Hirose_DM3AT-SF-PEJM5" H 12350 2450 50  0001 C CNN
 F 3 "https://www.hirose.com/product/en/download_file/key_name/DM3/category/Catalog/doc_file_id/49662/?file_category_id=4&item_id=195&is_series=1" H 10300 1850 50  0001 C CNN
-F 4 "秋月電子" H 10300 1750 50  0001 C CNN "Agency"
+F 4 "akizuki" H 10300 1750 50  0001 C CNN "Agency"
 F 5 "DM3AT-SF-PEJM5" H 10300 1750 50  0001 C CNN "MPN"
 F 6 "http://akizukidenshi.com/catalog/g/gC-02395/" H 10300 1750 50  0001 C CNN "Link"
@@
 F 2 "Diode_SMD:D_TUMD2" V 2900 4350 50  0001 C CNN
 F 3 "http://akizukidenshi.com/download/ds/rohm/rsx101vam30-j.pdf" V 2900 4350 50  0001 C CNN
-F 4 "秋月電子" H 2900 4350 50  0001 C CNN "Agency"
+F 4 "akizuki" H 2900 4350 50  0001 C CNN "Agency"
 F 5 "http://akizukidenshi.com/catalog/g/gI-05951/" H 2900 4350 50  0001 C CNN "Link"
 F 6 "RSX101VAM-30TR" H 2900 4350 50  0001 C CNN "MPN"
@@
 	1700 3650 1700 4200
 $Comp
-L power:VCC #PWR?
+L power:VCC #PWR0157
 U 1 1 5DBF619F
 P 1250 4200
-F 0 "#PWR?" H 1250 4050 50  0001 C CNN
+F 0 "#PWR0157" H 1250 4050 50  0001 C CNN
 F 1 "VCC" H 1267 4373 50  0000 C CNN
 F 2 "" H 1250 4200 50  0001 C CNN
@@
 Connection ~ 1250 4450
 $Comp
-L power:GND #PWR?
+L power:GND #PWR0158
 U 1 1 5DCA69C1
 P 700 4700
-F 0 "#PWR?" H 700 4450 50  0001 C CNN
+F 0 "#PWR0158" H 700 4450 50  0001 C CNN
 F 1 "GND" H 705 4527 50  0000 C CNN
 F 2 "" H 700 4700 50  0001 C CNN
